Commit message: Correct rotation angles, correct effort, remove dynamic friction and damping causing too slow motions

File: urdf/youbot_arm/arm.urdf.xacro (robot description, xacro)
@@ -39,16 +39,16 @@
 		<!-- joint between arm_0_link and arm_1_link -->
 		<joint name="${name}_joint_1" type="revolute">
-			<origin xyz="0.024 0 0.096" rpy="0 0 ${170 * M_PI / 180}"/>
+			<origin xyz="0.024 0 0.096" rpy="0 0 0"/>
 			<parent link="${name}_link_0"/>
 			<child link="${name}_link_1"/>
-			<axis xyz="0 0 -1"/>
+			<axis xyz="0 0 1"/>
 			<!--<calibration rising="${arm_1_ref}" falling="${arm_1_ref}"/>-->
-			<dynamics damping="1" friction="1" />
+<!--			<dynamics damping="1" friction="1" />-->
 			<!-- damping - N*s/m, N*s*m/rad -->
 			<!-- friction - N, N*m -->
-			<limit effort="${9.5}" velocity="${M_PI / 2.0}" lower="0" upper="${joint_1_limit}"/>
+			<limit effort="${joint_effort_1}" velocity="${M_PI / 2.0}" lower="${joint_1_limit_lower}" upper="${joint_1_limit_upper}"/>
 			<!--effort - N, N*m-->
 			<!--velocity - m/s, rad/s-->
-			<safety_controller k_position="20" k_velocity="${9.5/M_PI / 2.0}" soft_lower_limit="${threshold}" soft_upper_limit="${joint_1_limit_soft}" />
+<!--			<safety_controller k_position="20" k_velocity="${9.5/M_PI / 2.0}" soft_lower_limit="${threshold}" soft_upper_limit="${joint_1_limit_soft}" />-->
 			<!--k_position N/m, N/rad-->
 			<!--k_velocity N*s/m, N*s*m/rad-->
@@ -78,12 +78,12 @@
 		<!-- joint between arm_1_link and arm_2_link -->
 		<joint name="${name}_joint_2" type="revolute">
-			<origin xyz="0.033 0 0.019" rpy="0 ${-65 * M_PI / 180} 0"/>
+			<origin xyz="0.033 0 0.019" rpy="0 0 0"/>
 			<parent link="${name}_link_1"/>
 			<child link="${name}_link_2"/>
 			<axis xyz="0 1 0"/>
 			<!--<calibration rising="${arm_2_ref}" falling="${arm_2_ref}"/>-->
-			<dynamics damping="1" friction="1" />
-			<limit effort="${9.5}" velocity="${M_PI / 2.0}" lower="0" upper="${joint_2_limit}"/>
-                        <safety_controller k_position="20" k_velocity="${2*9.5/M_PI}" soft_lower_limit="${threshold}" soft_upper_limit="${joint_2_limit_soft}" />
+<!--			<dynamics damping="1" friction="1" />-->
+			<limit effort="${joint_effort_2}" velocity="${M_PI / 2.0}" lower="${joint_2_limit_lower}" upper="${joint_2_limit_upper}"/>
+<!--			<safety_controller k_position="20" k_velocity="${2*9.5/M_PI}" soft_lower_limit="${threshold}" soft_upper_limit="${joint_2_limit_soft}" />-->
 		</joint>
 		<link name="${name}_link_2">
@@ -119,11 +119,11 @@
 		</joint>-->
 		<joint name="${name}_joint_3" type="revolute">
-			<origin xyz="0.000 0.000 0.155" rpy="0 ${146 * M_PI / 180} 0"/>
+			<origin xyz="0.000 0.000 0.155" rpy="0 0 0"/>
 			<parent link="${name}_link_2"/>
 			<child link="${name}_link_3"/>
 			<axis xyz="0 1 0"/>
-			<dynamics damping="1" friction="1" />
-			<limit effort="${6}" velocity="${M_PI / 2.0}" lower="-${joint_3_limit}" upper="0"/>
-                        <safety_controller k_position="20" k_velocity="50" soft_lower_limit="-${joint_3_limit_soft}" soft_upper_limit="-${threshold}" />
+<!--			<dynamics damping="1" friction="1" />-->
+			<limit effort="${joint_effort_3}" velocity="${M_PI / 2.0}" lower="${joint_3_limit_lower}" upper="${joint_3_limit_upper}"/>
+<!--			<safety_controller k_position="20" k_velocity="50" soft_lower_limit="-${joint_3_limit_soft}" soft_upper_limit="-${threshold}" />-->
 		</joint>
 		<link name="${name}_link_3">
@@ -150,12 +150,12 @@
 		<!-- joint between arm_3_link and arm_4_link -->
 		<joint name="${name}_joint_4" type="revolute">
-			<origin xyz="0.000 0.000 0.135" rpy="0 ${-102.5 * M_PI / 180} 0" />
+			<origin xyz="0.000 0.000 0.135" rpy="0 0 0" />
 			<parent link="${name}_link_3"/>
 			<child link="${name}_link_4"/>
 			<axis xyz="0 1 0" />
 			<!--<calibration rising="${arm_4_ref}" falling="${arm_4_ref}"/>-->
-			<dynamics damping="1" friction="1" />
-			<limit effort="${2}" velocity="${M_PI / 2.0}" lower="0" upper="${joint_4_limit}"/>
-			<safety_controller k_position="20" k_velocity="100" soft_lower_limit="0" soft_upper_limit="${joint_4_limit_soft}" />
+<!--			<dynamics damping="1" friction="1" />-->
+			<limit effort="${joint_effort_4}" velocity="${M_PI / 2.0}" lower="${joint_4_limit_lower}" upper="${joint_4_limit_upper}"/>
+<!--			<safety_controller k_position="20" k_velocity="100" soft_lower_limit="0" soft_upper_limit="${joint_4_limit_soft}" />-->
 		</joint>
 		<link name="${name}_link_4">
@@ -182,12 +182,12 @@
 		<!-- joint between arm_4_link and arm_5_link -->
 		<joint name="${name}_joint_5" type="revolute">
-			<origin xyz="-0.002 0 0.130" rpy="0 0 ${167.5 * M_PI / 180}" />
+			<origin xyz="-0.002 0 0.130" rpy="0 0 0" />
 			<parent link="${name}_link_4"/>
 			<child link="${name}_link_5"/>
 			<axis xyz="0 0 -1" />
 			<!--<calibration rising="${arm_5_ref}" falling="${arm_5_ref}"/>-->
-			<dynamics damping="1" friction="1" />
-			<limit effort="1" velocity="${M_PI / 2.0}" lower="0" upper="${joint_5_limit}" />
-                        <safety_controller k_position="20" k_velocity="100" soft_lower_limit="0" soft_upper_limit="${joint_5_limit_soft}" />
+<!--			<dynamics damping="1" friction="1" />-->
+			<limit effort="${joint_effort_5}" velocity="${M_PI / 2.0}" lower="${joint_5_limit_lower}" upper="${joint_5_limit_upper}" />
+<!--			<safety_controller k_position="20" k_velocity="100" soft_lower_limit="0" soft_upper_limit="${joint_5_limit_soft}" />-->
 		</joint>
 		<link name="${name}_link_5">

File: urdf/youbot_arm/limits.urdf.xacro (robot description, xacro)
@@ -2,17 +2,22 @@
 <robot xmlns:xacro="http://ros.org/wiki/xacro">>
 	<!-- common properties -->
-	<xacro:property name="M_PI" value="3.1415926535897931" />
-        <xacro:property name="threshold" value="0.01" />
+	<xacro:property name="M_PI" value="3.1415926535897932" />
+	<xacro:property name="threshold" value="0.01" />
 	<!-- arm limits positions (deg) -->
-	<xacro:property name="joint_1_limit" value="${M_PI * (169 + 169) / 180}" />
-	<xacro:property name="joint_2_limit" value="${M_PI * (90 + 65) / 180}" />
-	<xacro:property name="joint_3_limit" value="${M_PI * (146 + 151) / 180}" />
-	<xacro:property name="joint_4_limit" value="${M_PI * (102.5 + 102.5) / 180}" />
-	<xacro:property name="joint_5_limit" value="${M_PI * (167.5 + 167.5) / 180}" />
-        <xacro:property name="joint_1_limit_soft" value="${M_PI * (169 + 169) / 180 - threshold}" />
-	<xacro:property name="joint_2_limit_soft" value="${M_PI * (90 + 65) / 180 - threshold}" />
-	<xacro:property name="joint_3_limit_soft" value="${M_PI * (146 + 151) / 180 - threshold}" />
-	<xacro:property name="joint_4_limit_soft" value="${M_PI * (102.5 + 102.5) / 180 - threshold}" />
-	<xacro:property name="joint_5_limit_soft" value="${M_PI * (167.5 + 167.5) / 180 - threshold}" />
+	<xacro:property name="joint_1_limit_lower" value="${M_PI * -169 /180}" />
+    <xacro:property name="joint_1_limit_upper" value="${M_PI * 169 /180}" />
+	<xacro:property name="joint_2_limit_lower" value="${M_PI * -65 /180}" />
+    <xacro:property name="joint_2_limit_upper" value="${M_PI * 90 /180}" />
+	<xacro:property name="joint_3_limit_lower" value="${M_PI * -146 /180}" />
+    <xacro:property name="joint_3_limit_upper" value="${M_PI * 150 /180}" />
+	<xacro:property name="joint_4_limit_lower" value="${M_PI * -102.5 /180}" />
+    <xacro:property name="joint_4_limit_upper" value="${M_PI * 102.5 /180}" />
+	<xacro:property name="joint_5_limit_lower" value="${M_PI * -167.5 /180}" />
+	<xacro:property name="joint_5_limit_upper" value="${M_PI * 167.5 /180}" />
+	<xacro:property name="joint_effort_1" value="${82.7 * 156 / 1000}" />
+	<xacro:property name="joint_effort_2" value="${82.7 * 156 / 1000}" />
+	<xacro:property name="joint_effort_3" value="${82.7 * 100 / 1000}" />
+	<xacro:property name="joint_effort_4" value="${58.8 * 71 / 1000}" />
+	<xacro:property name="joint_effort_5" value="${58.8 * 71 / 1000}" />
 	<!-- dynamic properties : mass (kg) Alu data sheet -->
 	<xacro:property name="link_0_mass" value="0.845" />
