Commit message: Multiply effort of arm joints to be able to reach normal velocities

File: urdf/youbot_arm/limits.urdf.xacro (robot description, xacro)
@@ -15,9 +15,9 @@
 	<xacro:property name="joint_5_limit_lower" value="${M_PI * -167.5 /180}" />
 	<xacro:property name="joint_5_limit_upper" value="${M_PI * 167.5 /180}" />
-	<xacro:property name="joint_effort_1" value="${82.7 * 156 / 1000}" />
-	<xacro:property name="joint_effort_2" value="${82.7 * 156 / 1000}" />
-	<xacro:property name="joint_effort_3" value="${82.7 * 100 / 1000}" />
-	<xacro:property name="joint_effort_4" value="${58.8 * 71 / 1000}" />
-	<xacro:property name="joint_effort_5" value="${58.8 * 71 / 1000}" />
+	<xacro:property name="joint_effort_1" value="${4 * 82.7 * 156 / 1000}" />
+	<xacro:property name="joint_effort_2" value="${4 * 82.7 * 156 / 1000}" />
+	<xacro:property name="joint_effort_3" value="${4 * 82.7 * 100 / 1000}" />
+	<xacro:property name="joint_effort_4" value="${4 * 58.8 * 71 / 1000}" />
+	<xacro:property name="joint_effort_5" value="${4 * 58.8 * 71 / 1000}" />
 	<!-- dynamic properties : mass (kg) Alu data sheet -->
 	<xacro:property name="link_0_mass" value="0.845" />

Commit message: Multiply effort to make the arm stronger

File: urdf/youbot_arm/limits.urdf.xacro (robot description, xacro)
@@ -4,4 +4,5 @@
 	<xacro:property name="M_PI" value="3.1415926535897932" />
 	<xacro:property name="threshold" value="0.01" />
+	<xacro:property name="effort_multiplier" value="10" />
 	<!-- arm limits positions (deg) -->
 	<xacro:property name="joint_1_limit_lower" value="${M_PI * -169 /180}" />
@@ -15,9 +16,9 @@
 	<xacro:property name="joint_5_limit_lower" value="${M_PI * -167.5 /180}" />
 	<xacro:property name="joint_5_limit_upper" value="${M_PI * 167.5 /180}" />
-	<xacro:property name="joint_effort_1" value="${4 * 82.7 * 156 / 1000}" />
-	<xacro:property name="joint_effort_2" value="${4 * 82.7 * 156 / 1000}" />
-	<xacro:property name="joint_effort_3" value="${4 * 82.7 * 100 / 1000}" />
-	<xacro:property name="joint_effort_4" value="${4 * 58.8 * 71 / 1000}" />
-	<xacro:property name="joint_effort_5" value="${4 * 58.8 * 71 / 1000}" />
+	<xacro:property name="joint_effort_1" value="${effort_multiplier * 82.7 * 156 / 1000}" />
+	<xacro:property name="joint_effort_2" value="${effort_multiplier * 82.7 * 156 / 1000}" />
+	<xacro:property name="joint_effort_3" value="${effort_multiplier * 82.7 * 100 / 1000}" />
+	<xacro:property name="joint_effort_4" value="${effort_multiplier * 58.8 * 71 / 1000}" />
+	<xacro:property name="joint_effort_5" value="${effort_multiplier * 58.8 * 71 / 1000}" />
 	<!-- dynamic properties : mass (kg) Alu data sheet -->
 	<xacro:property name="link_0_mass" value="0.845" />

Commit message: Edit arm effort

File: urdf/youbot_arm/limits.urdf.xacro (robot description, xacro)
@@ -16,9 +16,9 @@
 	<xacro:property name="joint_5_limit_lower" value="${M_PI * -167.5 /180}" />
 	<xacro:property name="joint_5_limit_upper" value="${M_PI * 167.5 /180}" />
-	<xacro:property name="joint_effort_1" value="${effort_multiplier * 82.7 * 156 / 1000}" />
-	<xacro:property name="joint_effort_2" value="${effort_multiplier * 82.7 * 156 / 1000}" />
-	<xacro:property name="joint_effort_3" value="${effort_multiplier * 82.7 * 100 / 1000}" />
-	<xacro:property name="joint_effort_4" value="${effort_multiplier * 58.8 * 71 / 1000}" />
-	<xacro:property name="joint_effort_5" value="${effort_multiplier * 58.8 * 71 / 1000}" />
+	<xacro:property name="joint_effort_1" value="${effort_multiplier * 9.5}" />
+	<xacro:property name="joint_effort_2" value="${effort_multiplier * 9.5}" />
+	<xacro:property name="joint_effort_3" value="${effort_multiplier * 6.0}" />
+	<xacro:property name="joint_effort_4" value="${effort_multiplier * 2.0}" />
+	<xacro:property name="joint_effort_5" value="${effort_multiplier * 1.0}" />
 	<!-- dynamic properties : mass (kg) Alu data sheet -->
 	<xacro:property name="link_0_mass" value="0.845" />

Commit message: Revert "Edit arm effort"
This reverts commit 9b0a1686d1cb5cc719ace748c0b7215402061e12.

File: urdf/youbot_arm/limits.urdf.xacro (robot description, xacro)
@@ -16,9 +16,9 @@
 	<xacro:property name="joint_5_limit_lower" value="${M_PI * -167.5 /180}" />
 	<xacro:property name="joint_5_limit_upper" value="${M_PI * 167.5 /180}" />
-	<xacro:property name="joint_effort_1" value="${effort_multiplier * 9.5}" />
-	<xacro:property name="joint_effort_2" value="${effort_multiplier * 9.5}" />
-	<xacro:property name="joint_effort_3" value="${effort_multiplier * 6.0}" />
-	<xacro:property name="joint_effort_4" value="${effort_multiplier * 2.0}" />
-	<xacro:property name="joint_effort_5" value="${effort_multiplier * 1.0}" />
+	<xacro:property name="joint_effort_1" value="${effort_multiplier * 82.7 * 156 / 1000}" />
+	<xacro:property name="joint_effort_2" value="${effort_multiplier * 82.7 * 156 / 1000}" />
+	<xacro:property name="joint_effort_3" value="${effort_multiplier * 82.7 * 100 / 1000}" />
+	<xacro:property name="joint_effort_4" value="${effort_multiplier * 58.8 * 71 / 1000}" />
+	<xacro:property name="joint_effort_5" value="${effort_multiplier * 58.8 * 71 / 1000}" />
 	<!-- dynamic properties : mass (kg) Alu data sheet -->
 	<xacro:property name="link_0_mass" value="0.845" />
