Commit message: Add nice looking wheels

File: urdf/youbot_base/base.urdf.xacro (robot description, xacro)
@@ -115,5 +115,5 @@
         <!--<mesh filename="package://youbot_description/meshes/youbot_base/youbot_wheel.stl" />-->
         <geometry>
-          <sphere radius="${wheel_radius}"/>
+          <mesh filename="package://youbot_description/meshes/youbot_base/front-left_wheel.dae"/>
         </geometry>
         <material name="Orange"/>
@@ -161,6 +161,5 @@
         <origin xyz="0 0 0" rpy="0 0 0"/>
         <geometry>
-          <!--<mesh filename="package://youbot_description/meshes/youbot_base/youbot_wheel.stl" />-->
-          <sphere radius="${wheel_radius}"/>
+          <mesh filename="package://youbot_description/meshes/youbot_base/front-right_wheel.dae"/>
         </geometry>
         <material name="Orange"/>
@@ -209,6 +208,5 @@
         <origin xyz="0 0 0" rpy="0 0 0"/>
         <geometry>
-          <!--<mesh filename="package://youbot_description/meshes/youbot_base/youbot_wheel.stl" />-->
-          <sphere radius="${wheel_radius}"/>
+          <mesh filename="package://youbot_description/meshes/youbot_base/back-left_wheel.dae"/>
         </geometry>
         <material name="Orange"/>
@@ -256,6 +254,5 @@
         <origin xyz="0 0 0" rpy="0 0 0"/>
         <geometry>
-          <!--<mesh filename="package://youbot_description/meshes/youbot_base/youbot_wheel.stl" />-->
-          <sphere radius="${wheel_radius}"/>
+          <mesh filename="package://youbot_description/meshes/youbot_base/back-right_wheel.dae"/>
         </geometry>
         <material name="Orange"/>
